Commit message: Add rviz config file and material color.

File: urdf/mys450f_macro.xacro (robot description, xacro)
@@ -13,4 +13,8 @@
   <xacro:property name="acc" value="20"/>
   <xacro:macro name="motoman_mys450f" params="prefix">
+    <!-- Properties -->
+    <material name="yaskawa_blue">
+      <color rgba="0.12941 0.14902 0.74902 1" />
+    </material>
     <!-- link list -->
     <link name="${prefix}base_link">
@@ -19,4 +23,7 @@
           <mesh filename="package://motoman_mys450f_support/meshes/mys450f/visual/base_link.dae"/>
         </geometry>
+        <material name="white">
+          <color rgba="0.7 0.7 0.7 1.0"/>
+        </material>
       </visual>
       <collision>
@@ -39,4 +46,5 @@
           <mesh filename="package://motoman_mys450f_support/meshes/mys450f/visual/link_1_s.dae"/>
         </geometry>
+        <material name="yaskawa_blue"/>
       </visual>
       <collision>
@@ -59,4 +67,7 @@
           <mesh filename="package://motoman_mys450f_support/meshes/mys450f/visual/link_2_l.dae"/>
         </geometry>
+        <material name="grey">
+          <color rgba="0.3 0.3 0.3 1.0"/>
+        </material>
       </visual>
       <collision>
@@ -79,4 +90,7 @@
           <mesh filename="package://motoman_mys450f_support/meshes/mys450f/visual/link_3_u.dae"/>
         </geometry>
+        <material name="black">
+          <color rgba="0.1 0.1 0.1 1.0"/>
+        </material>
       </visual>
       <collision>

Commit message: change visual mesh from dae to stl and update material color

File: urdf/mys450f_macro.xacro (robot description, xacro)
@@ -17,13 +17,20 @@
       <color rgba="0.12941 0.14902 0.74902 1" />
     </material>
+    <material name="white">
+      <color rgba="1.0 1.0 1.0 1.0"/>
+    </material>
+    <material name="grey">
+      <color rgba="0.4 0.4 0.4 1.0"/>
+    </material>
+    <material name="silver">
+      <color rgba="0.6 0.6 0.6 1.0"/>
+    </material>
     <!-- link list -->
     <link name="${prefix}base_link">
       <visual>
         <geometry>
-          <mesh filename="package://motoman_mys450f_support/meshes/mys450f/visual/base_link.dae"/>
+          <mesh filename="package://motoman_mys450f_support/meshes/mys450f/visual/base_link.stl"/>
         </geometry>
-        <material name="white">
-          <color rgba="0.7 0.7 0.7 1.0"/>
-        </material>
+        <material name="white"/>
       </visual>
       <collision>
@@ -44,5 +51,5 @@
       <visual>
         <geometry>
-          <mesh filename="package://motoman_mys450f_support/meshes/mys450f/visual/link_1_s.dae"/>
+          <mesh filename="package://motoman_mys450f_support/meshes/mys450f/visual/link_1_s.stl"/>
         </geometry>
         <material name="yaskawa_blue"/>
@@ -65,9 +72,7 @@
       <visual>
         <geometry>
-          <mesh filename="package://motoman_mys450f_support/meshes/mys450f/visual/link_2_l.dae"/>
+          <mesh filename="package://motoman_mys450f_support/meshes/mys450f/visual/link_2_l.stl"/>
         </geometry>
-        <material name="grey">
-          <color rgba="0.3 0.3 0.3 1.0"/>
-        </material>
+        <material name="white"/>
       </visual>
       <collision>
@@ -88,9 +93,7 @@
       <visual>
         <geometry>
-          <mesh filename="package://motoman_mys450f_support/meshes/mys450f/visual/link_3_u.dae"/>
+          <mesh filename="package://motoman_mys450f_support/meshes/mys450f/visual/link_3_u.stl"/>
         </geometry>
-        <material name="black">
-          <color rgba="0.1 0.1 0.1 1.0"/>
-        </material>
+        <material name="silver"/>
       </visual>
       <collision>

Commit message: Add Yaskawa logo on link2_l

File: urdf/mys450f_macro.xacro (robot description, xacro)
@@ -112,4 +112,20 @@
     </link>
     <link name="${prefix}tool0"/>
+    <link name="${prefix}logo_f">
+      <visual>
+        <geometry>
+          <mesh filename="package://motoman_mys450f_support/meshes/mys450f/visual/logo.stl" scale="1.0 1.0 1.2"/>
+        </geometry>
+        <material name="yaskawa_blue"/>
+      </visual>
+    </link>
+    <link name="${prefix}logo_b">
+      <visual>
+        <geometry>
+          <mesh filename="package://motoman_mys450f_support/meshes/mys450f/visual/logo.stl" scale="1.0 1.0 1.2"/>
+        </geometry>
+        <material name="yaskawa_blue"/>
+      </visual>
+    </link>
     <!-- end of link list -->
     <!-- joint list -->
@@ -146,19 +162,16 @@
       <dynamics damping="0.7"/>
     </joint>
-    <!--
-    <joint name="${prefix}joint_4_r" type="revolute">
+    <joint name="${prefix}joint_2_l-logo_f" type="fixed">
       <parent link="${prefix}link_2_l"/>
-      <child link="${prefix}link_3_u"/>
-      <origin xyz="0.0 0.0 0.0" rpy="0 0 0"/>
-      <axis xyz="0 0 -1"/>
-      <limit lower="${-360.0*deg}" upper="${360.0*deg}" effort="${acc*deg}" velocity="${acc*deg}"/>
-      <dynamics damping="0.7"/>
+      <child link="${prefix}logo_f"/>
+      <origin xyz="0.185 0.05 0.12" rpy="0 0 0"/>
+      <axis xyz="0 0 1"/>
     </joint>
-    <joint name="${prefix}joint_4_r-tool0" type="fixed">
-      <parent link="${prefix}link_3_u"/>
-      <child link="${prefix}tool0"/>
-      <origin xyz="0.0 0.0 0.0" rpy="0 0 0"/>
+    <joint name="${prefix}joint_2_l-logo_b" type="fixed">
+      <parent link="${prefix}link_2_l"/>
+      <child link="${prefix}logo_b"/>
+      <origin xyz="0.060 -0.05 0.12" rpy="0 0 ${180.0*deg}"/>
+      <axis xyz="0 0 1"/>
     </joint>
-    -->
     <!-- end of joint list -->
     <!-- ROS base_link to Motoman World Coordinates transform -->
